File: KiPad.kicad_sch (KiCad schematic)
At the start: 0 parts

Commit message: schematic and assigned footprints done
Parts:
- added D1, D10, D11, D12, D2, D3, D4, D5, D6, D7, D8, D9: 1N4148, Diode_THT:D_DO-35_SOD27_P7.62mm_Horizontal, symbol Diode:1N4148
- added SW1, SW10, SW11, SW12, SW2, SW3, SW4, SW5, SW6, SW7, SW8, SW9: SW_Push_45deg, Button_Switch_Keyboard:SW_Cherry_MX_1.00u_PCB, symbol Switch:SW_Push_45deg
- added U1: XIAO-RP2040-DIP, Module:MOUDLE14P-XIAO-DIP-SMD, symbol Seeed_Studio_XIAO_Series:XIAO-RP2040-DIP
Connections:
- new net: D11.2 (A), SW11.2
- new net: D3.2 (A), SW3.2
- new net: D5.2 (A), SW5.2
- new net: D6.2 (A), SW6.2
- new net: D8.2 (A), SW8.2
- new net: D4.2 (A), SW4.2
- new net: D2.2 (A), SW2.2
- new net: D1.2 (A), SW1.2
- new net: D7.2 (A), SW7.2
- new net: D12.2 (A), SW12.2
- new net: D10.2 (A), SW10.2
- new net: D9.2 (A), SW9.2
- new net COL1: D1.1 (K), D10.1 (K), D4.1 (K), D7.1 (K), U1.5 (GPIO6/SDA)
- new net COL2: D11.1 (K), D2.1 (K), D5.1 (K), D8.1 (K), U1.6 (GPIO7/SCL)
- new net COL3: D12.1 (K), D3.1 (K), D6.1 (K), D9.1 (K), U1.7 (GPIO0/TX)
- new net ROW1: SW1.1, SW2.1, SW3.1, U1.1 (GPIO26/ADC0/A0)
- new net ROW2: SW4.1, SW5.1, SW6.1, U1.2 (GPIO27/ADC1/A1)
- new net ROW3: SW7.1, SW8.1, SW9.1, U1.3 (GPIO28/ADC2/A2)
- new net ROW4: SW10.1, SW11.1, SW12.1, U1.4 (GPIO29/ADC3/A3)

Commit message: finished pcb design
Parts:
- U1: footprint Module:MOUDLE14P-XIAO-DIP-SMD -> footprints:XIAO-RP2040-DIP
Changed lines of the file:
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@@
 			)
 		)
-		(property "Footprint" "Module:MOUDLE14P-XIAO-DIP-SMD"
+		(property "Footprint" "footprints:XIAO-RP2040-DIP"
 			(at 104.648 107.188 0)
 			(hide yes)
